File: hardware/keg-module-pcb/keg_sensor_module.kicad_sch (KiCad schematic)
At the start: 7 parts, among them J1 Sensor_FL, J2 Sensor_FR, J3 Sensor_BR, J4 Sensor_BL, J5 HX711_LoadCell_Side, J6 HX711_Digital_Side, J7 RJ11_to_Hub

Commit message: Brand project as Sallaup Electronics / KegSensor (Sallaup KegSense system)
Schematic title block, docs, and case.scad header updated. Regenerated
schematic + PDF, re-ran ERC to confirm still clean.
Other:
- company: (none) -> Sallaup Electronics
- title: Keg Sensor Module -> KegSensor
