File: hardware/keg-module-pcb/keg_sensor_module.kicad_pcb (KiCad board)
At the start: 2 copper layers, 155 x 90 mm, 11 parts, among them J1 TerminalBlock_bornier-3_P5.08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, J2 TerminalBlock_bornier-3_P5.08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, J3 TerminalBlock_bornier-3_P5.08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, J4 TerminalBlock_bornier-3_P5.08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, J5 PinSocket_1x04_P2.54mm_Vertic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, J6 PinSocket_1x04_P2.54mm_Vertic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, J7 RJ14_Connfly_DS1133-S4_Horizo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

Commit message: Fix J7 (RJ11 jack) reachability: move to board edge, rewire, fix case cutout
J7 was placed mid-board with no path to any wall (13.7mm from the right
wall, 27mm from the top wall) - the case's cutout, built assuming it was
near the top edge, didn't align with it at all. Root cause was a stale
board outline value (145mm instead of 155mm) left over from before the
mounting holes were added, which also caused knock-on edge-clearance
DRC errors once J7 moved.

Fix: rotate J7 -90deg and move it flush with the board's right edge (the
correct placement for any edge connector, independent of the case),
rewrite the J6<->J7 routing for the new pad positions, fix the stale
outline, and move the case's cutout from the top wall to the right wall
at J7's actual position. Along the way, confirmed empirically (via DRC's
reported pad coordinates, not assumption) that KiCad's footprint rotation
is the opposite sign of the standard math convention - same class of bug
as the earlier schematic Y-axis surprise.

DRC: 0 errors (2 cosmetic warnings: silkscreen slightly clipped by the
board edge for an edge-mounted connector, and a footprint metadata diff
from the property-stripping in generate_pcb.py - neither electrical).
Parts:
- removed MH1, MH2, MH3, MH4: MountingHole_3.2mm_M3, MountingHole:MountingHole_3.2mm_M3
- moved J7 11.2 mm to (146.0, 35.0), turned to -90 degrees
Routing:
- net VCC_3V3: track 60.1 -> 107.1 mm, vias 0 -> 2
- net GND: track 42.0 -> 81.0 mm, vias 0 -> 1
- net DT: track 53.1 -> 72.9 mm, vias 0 -> 1
- net SCK: track 65.1 -> 77.9 mm

Commit message: Add KegSensor / Sallaup Electronics branding to the PCB silkscreen
First placement (30,58) overlapped J2/J4's reference-label silkscreen -
DRC caught it (silk_overlap warnings), repositioned into the clear gap
between J2 and J4 and re-verified DRC comes back clean (down to the same
2 pre-existing cosmetic warnings as before: J7's silkscreen slightly
clipped by the board edge, and a footprint-metadata diff, neither
electrical).
Other:
- board text added: "KegSensor"
- board text added: "Sallaup Electronics"
Changed lines of the file:
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@@
 		(net 8)
+	)
+	(gr_text "KegSensor"
+		(at 26 63 0)
+		(layer "F.SilkS")
+		(effects
+			(font
+				(size 2.2 2.2)
+				(thickness 0.33)
+			)
+		)
+	)
+	(gr_text "Sallaup Electronics"
+		(at 26 67 0)
+		(layer "F.SilkS")
+		(effects
+			(font
+				(size 1.2 1.2)
+				(thickness 0.18)
+			)
+		)
 	)
 	(embedded_fonts no)

Commit message: Add Rev A / 2026 to the PCB silkscreen
Placed in the open area right of J5/below the J6<->J7 routing (that
routing stays y<=52; nothing else occupies x=60-155, y=52-90). DRC still
clean (same 2 pre-existing cosmetic warnings, no new overlaps).
Other:
- board text added: "2026"
- board text added: "Rev A"
Changed lines of the file:
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@@
+		)
+	)
+	(gr_text "Rev A"
+		(at 100 68 0)
+		(layer "F.SilkS")
+		(effects
+			(font
+				(size 2.2 2.2)
+				(thickness 0.33)
+			)
+		)
+	)
+	(gr_text "2026"
+		(at 100 72 0)
+		(layer "F.SilkS")
+		(effects
+			(font
+				(size 1.5 1.5)
+				(thickness 0.225)
+			)
 		)
 	)
