File: hardware/kegsensor/keg_sensor_module.kicad_pcb (KiCad board)
At the start: 2 copper layers, 155 x 90 mm, 7 parts, among them J1 TerminalBlock_bornier-3_P5.08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, J2 TerminalBlock_bornier-3_P5.08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, J3 TerminalBlock_bornier-3_P5.08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, J4 TerminalBlock_bornier-3_P5.08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, J5 PinSocket_1x04_P2.54mm_Vertic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, J6 PinSocket_1x04_P2.54mm_Vertic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, J7 RJ14_Connfly_DS1133-S4_Horizo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

Commit message: Simplify J6-J7 routing: single layer per net where possible
Each of GND/VCC/SCK/DT previously had a short F.Cu stub off J6 before
via-ing to B.Cu for the rest, on every net - vestigial for two of them.
GND and SCK are now a single unbroken line on one layer each (B.Cu and
F.Cu respectively), no vias - J6's pads are through-hole, so a track
can start on whichever layer it needs directly at the pad.

VCC_3V3 and DT keep one via each - not a missed simplification but real
geometry, checked exhaustively rather than just patched around the
first conflict DRC caught: VCC's own source row at J6 sits inside DT's
drop's depth range, and DT's row sits inside VCC's, so whichever one is
in the way at that crossing needs to be on the other layer right there.
Two vias is the minimum for this connector, down from four.

DRC clean (1 pre-existing accepted warning). Regenerated fab/ Gerbers,
drill files, and PCB renders to match.

Co-Authored-By: Claude Sonnet 5 <noreply@anthropic.com>
Routing:
- net SCK: vias 2 -> 0
- net GND: vias 1 -> 0
Changed lines of the file:
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@@
 		(end 103 35)
 		(width 0.3)
-		(layer "F.Cu")
+		(layer "B.Cu")
 		(net 5)
 	)
@@
 	)
 	(segment
+		(start 95 40.08)
+		(end 102 40.08)
+		(width 0.3)
+		(layer "F.Cu")
+		(net 7)
+	)
+	(segment
+		(start 102 40.08)
+		(end 102 65)
+		(width 0.3)
+		(layer "F.Cu")
+		(net 7)
+	)
+	(segment
+		(start 102 65)
+		(end 140 65)
+		(width 0.3)
+		(layer "F.Cu")
+		(net 7)
+	)
+	(segment
+		(start 140 65)
+		(end 140 81)
+		(width 0.3)
+		(layer "F.Cu")
+		(net 7)
+	)
+	(segment
+		(start 140 81)
+		(end 143.96 81)
+		(width 0.3)
+		(layer "F.Cu")
+		(net 7)
+	)
+	(segment
 		(start 95 42.62)
 		(end 101 42.62)
@@
 	)
 	(segment
-		(start 95 40.08)
-		(end 99 40.08)
-		(width 0.3)
-		(layer "F.Cu")
-		(net 7)
-	)
-	(segment
-		(start 99 40.08)
-		(end 99 65)
-		(width 0.3)
-		(layer "B.Cu")
-		(net 7)
-	)
-	(segment
-		(start 99 65)
-		(end 140 65)
-		(width 0.3)
-		(layer "F.Cu")
-		(net 7)
-	)
-	(segment
-		(start 140 65)
-		(end 140 81)
-		(width 0.3)
-		(layer "F.Cu")
-		(net 7)
-	)
-	(segment
-		(start 140 81)
-		(end 143.96 81)
-		(width 0.3)
-		(layer "F.Cu")
-		(net 7)
-	)
-	(segment
 		(start 95 37.54)
 		(end 97 37.54)
@@
 	)
 	(via
-		(at 103 35)
-		(size 0.6)
-		(drill 0.3)
-		(layers "F.Cu" "B.Cu")
-		(net 5)
-	)
-	(via
 		(at 101 42.62)
 		(size 0.6)
@@
 	)
 	(via
-		(at 99 40.08)
-		(size 0.6)
-		(drill 0.3)
-		(layers "F.Cu" "B.Cu")
-		(net 7)
-	)
-	(via
-		(at 99 65)
-		(size 0.6)
-		(drill 0.3)
-		(layers "F.Cu" "B.Cu")
-		(net 7)
-	)
-	(via

Commit message: Silkscreen R/B/W wire-color labels above J1-J4's pins
Prints "R B W" above each of J1-J4's 3 pins (pin1=R, pin2=B, pin3=W,
fixed order on every connector), matching the documented sensor lead
convention (wiring.md: Red=E+, Black=E-, White=Signal) - so wiring a
sensor by color doesn't need the README open next to the board.

Positioned above each connector, between the board edge and the
connector body, clear of both the edge and each connector's own
reference designator - verified via DRC (silk_overlap), not just
eyeballed. DRC clean (1 pre-existing accepted warning).

Regenerated fab/ Gerbers, drill files, and PCB renders to match.

Co-Authored-By: Claude Sonnet 5 <noreply@anthropic.com>
Other:
- board text added: "B"
- board text added: "R"
- board text added: "W"
Changed lines of the file:
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@@
 		(net 6)
+	)
+	(gr_text "R"
+		(at 20 3 0)
+		(layer "F.SilkS")
+		(effects
+			(font
+				(size 1.0 1.0)
+				(thickness 0.15)
+			)
+		)
+	)
+	(gr_text "B"
+		(at 25.08 3 0)
+		(layer "F.SilkS")
+		(effects
+			(font
+				(size 1.0 1.0)
+				(thickness 0.15)
+			)
+		)
+	)
+	(gr_text "W"
+		(at 30.16 3 0)
+		(layer "F.SilkS")
+		(effects
+			(font
+				(size 1.0 1.0)
+				(thickness 0.15)
+			)
+		)
+	)
+	(gr_text "R"
+		(at 50 3 0)
+		(layer "F.SilkS")
+		(effects
+			(font
+				(size 1.0 1.0)
+				(thickness 0.15)
+			)
+		)
+	)
+	(gr_text "B"
+		(at 55.08 3 0)
+		(layer "F.SilkS")
+		(effects
+			(font
+				(size 1.0 1.0)
+				(thickness 0.15)
+			)
+		)
+	)
+	(gr_text "W"
+		(at 60.16 3 0)
+		(layer "F.SilkS")
+		(effects
+			(font
+				(size 1.0 1.0)
+				(thickness 0.15)
+			)
+		)
+	)
+	(gr_text "R"
+		(at 80 3 0)
+		(layer "F.SilkS")
+		(effects
+			(font
+				(size 1.0 1.0)
+				(thickness 0.15)
+			)
+		)
+	)
+	(gr_text "B"
+		(at 85.08 3 0)
+		(layer "F.SilkS")
+		(effects
+			(font
+				(size 1.0 1.0)
+				(thickness 0.15)
+			)
+		)
+	)
+	(gr_text "W"
+		(at 90.16 3 0)
+		(layer "F.SilkS")
+		(effects
+			(font
+				(size 1.0 1.0)
+				(thickness 0.15)
+			)
+		)
+	)
+	(gr_text "R"
+		(at 110 3 0)
+		(layer "F.SilkS")
+		(effects
+			(font
+				(size 1.0 1.0)
+				(thickness 0.15)
+			)
+		)
+	)
+	(gr_text "B"
+		(at 115.08 3 0)
+		(layer "F.SilkS")
+		(effects
+			(font
+				(size 1.0 1.0)
+				(thickness 0.15)
+			)
+		)
+	)
+	(gr_text "W"
+		(at 120.16 3 0)
+		(layer "F.SilkS")
+		(effects
+			(font
+				(size 1.0 1.0)
+				(thickness 0.15)
+			)
+		)
 	)
 	(gr_text "KegSensor"

Commit message: Silkscreen pin labels for J5/J6 (HX711 header)
E+/E-/A+/A- next to J5's pins, GND/DT/SCK/VCC next to J6's, matching the
Connectors table. Both are single-column vertical headers (4 pins
stacked at one X, 2.54mm pitch), so labels sit beside each pin rather
than above/below like J1-J4's row got. J6's needed extra clearance from
its own footprint outline - the 3-character labels clipped it at the
first attempt (DRC: silk_overlap), fixed by pushing them out further.

DRC clean (1 pre-existing accepted warning). Regenerated fab/ Gerbers,
drill files, and PCB renders to match.

Co-Authored-By: Claude Sonnet 5 <noreply@anthropic.com>
Other:
- board text added: "A+"
- board text added: "A-"
- board text added: "DT"
- board text added: "E+"
- board text added: "E-"
- board text added: "GND"
- board text added: "SCK"
- board text added: "VCC"
Changed lines of the file:
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@@
+		)
+	)
+	(gr_text "E+"
+		(at 62.5 35.0 0)
+		(layer "F.SilkS")
+		(effects
+			(font
+				(size 0.9 0.9)
+				(thickness 0.135)
+			)
+		)
+	)
+	(gr_text "E-"
+		(at 62.5 37.54 0)
+		(layer "F.SilkS")
+		(effects
+			(font
+				(size 0.9 0.9)
+				(thickness 0.135)
+			)
+		)
+	)
+	(gr_text "A+"
+		(at 62.5 40.08 0)
+		(layer "F.SilkS")
+		(effects
+			(font
+				(size 0.9 0.9)
+				(thickness 0.135)
+			)
+		)
+	)
+	(gr_text "A-"
+		(at 62.5 42.62 0)
+		(layer "F.SilkS")
+		(effects
+			(font
+				(size 0.9 0.9)
+				(thickness 0.135)
+			)
+		)
+	)
+	(gr_text "GND"
+		(at 99.5 35.0 0)
+		(layer "F.SilkS")
+		(effects
+			(font
+				(size 0.9 0.9)
+				(thickness 0.135)
+			)
+		)
+	)
+	(gr_text "DT"
+		(at 99.5 37.54 0)
+		(layer "F.SilkS")
+		(effects
+			(font
+				(size 0.9 0.9)
+				(thickness 0.135)
+			)
+		)
+	)
+	(gr_text "SCK"
+		(at 99.5 40.08 0)
+		(layer "F.SilkS")
+		(effects
+			(font
+				(size 0.9 0.9)
+				(thickness 0.135)
+			)
+		)
+	)
+	(gr_text "VCC"
+		(at 99.5 42.62 0)
+		(layer "F.SilkS")
+		(effects
+			(font
+				(size 0.9 0.9)
+				(thickness 0.135)
+			)
 		)
 	)
